File: pcb/myfirst_keeb_pcb.kicad_pcb (KiCad board)
At the start: 2 copper layers, 320.9 x 111.1 mm, 164 parts, among them J1 Conn_ARM_JTAG_SWD_10, Q1 DTC123J, SW1 SW_Push, SW3 Rotary_Encoder_Switch, U1 SRV05-4, U2 MCP1700-3302E_SOT23, U3 STM32F411RETx

Commit message: switch stm32f11 to stm32f07 for usb crystal
Parts:
- removed C9: 4.7uF, Capacitor_SMD:C_0805_2012Metric
- added TP1: TestPoint, TestPoint:TestPoint_Pad_D2.0mm, F.Cu at (150.0, 92.0)
- added TP2: TestPoint, TestPoint:TestPoint_Pad_D2.0mm, F.Cu at (138.2, 91.2)
- added TP3: TestPoint, TestPoint:TestPoint_Pad_D2.0mm, F.Cu at (210.5, 121.5)
- added TP4: TestPoint, TestPoint:TestPoint_Pad_D2.0mm, F.Cu at (225.0, 122.2)
- U3: value STM32F411RETx -> STM32F072CBTx; footprint Package_QFP:LQFP-64_10x10mm_P0.5mm -> Package_QFP:LQFP-48_7x7mm_P0.5mm
Connections:
- net EXTRA_PIN_PC13 renamed Net-(U3-Pad2)
- net EXTRA_PIN_PC14 renamed Net-(U3-Pad3)
- net EXTRA_PIN_PC15 renamed Net-(U3-Pad4)
- net EXTRA_PIN_PH0 renamed Net-(U3-Pad5)
- net EXTRA_PIN_PH1 renamed Net-(U3-Pad6)
- U3 pad 12: GND -> ROW4
- U3 pad 13: +3V3 -> Net-(U3-Pad13)
- U3 pad 14: Net-(U3-Pad14) -> COL0
- U3 pad 15: Net-(U3-Pad15) -> COL1
- U3 pad 16: ROW4 -> COL2
- U3 pad 17: Net-(U3-Pad17) -> COL3
- U3 pad 18: GND -> ROW0
- U3 pad 19: +3V3 -> ROW1
- U3 pad 20: COL0 -> ROW2
- U3 pad 21: COL1 -> ROW3
- U3 pad 22: COL2 -> Net-(U3-Pad22)
- U3 pad 23: COL3 -> GND
- U3 pad 24: ROW0 -> +3V3
- U3 pad 25: ROW1 -> COL4
- U3 pad 26: ROW2 -> COL5
- U3 pad 27: ROW3 -> COL6
- U3 pad 28: Net-(U3-Pad28) -> COL7
- U3 pad 29: Net-(U3-Pad29) -> COL8
- U3 pad 30: Net-(C9-Pad1) -> COL9
- U3 pad 31: GND -> COL10
- U3 pad 32: +3V3 -> D-
- U3 pad 33: COL4 -> D+
- U3 pad 34: COL5 -> SWDIO
- U3 pad 35: COL6 -> GND
- U3 pad 36: COL7 -> +3V3
- U3 pad 37: COL8 -> SWDCLK
- U3 pad 38: COL9 -> COL11
- U3 pad 39: COL10 -> COL12
- U3 pad 40: Net-(U3-Pad40) -> COL13
- U3 pad 41: Net-(U3-Pad41) -> COL14
- U3 pad 44: D- -> BOOT0
- U3 pad 45: D+ -> ENCODER_A
- U3 pad 46: SWDIO -> ENCODER_B
- U3 pad 8: Net-(U3-Pad8) -> GND
- U3 pad 9: Net-(U3-Pad9) -> +3V3
Routing:
- net GND: track 333.8 -> 361.0 mm, vias 7 -> 11
- net NRST: track 71.1 -> 78.3 mm
- net D+: track 110.9 -> 117.6 mm
- net Net-(C9-Pad1): track 5.44 -> 0.00 mm, vias 2 -> 0
- net BOOT0: track 77.1 -> 82.3 mm
- net D-: track 111.3 -> 116.5 mm
- net +3V3: track 432.6 -> 428.3 mm
- net COL10: track 206.1 -> 208.3 mm
- net COL13: track 254.4 -> 256.5 mm
- net SWDIO: track 56.2 -> 58.2 mm
- net SWDCLK: track 58.5 -> 60.4 mm
- net ENCODER_A: track 269.0 -> 270.9 mm
- net COL9: track 192.1 -> 194.1 mm
- net COL8: track 140.1 -> 142.0 mm
- net COL7: track 122.3 -> 124.2 mm
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Other:
- board text added: "BOOT"
- board text added: "D+"
- board text added: "D-"
- board text added: "RST"
- board text added: "zap"
- board text removed: "Zap!"

Commit message: change to hotswap kalih switches
Parts:
- MX1, MX10, MX11, MX12, MX13, MX15, MX16, MX17, MX18, MX20, MX21, MX22, MX23, MX24, MX25, MX26, MX27, MX28, MX29, MX30, MX31, MX33, MX34, MX35, MX36, MX37, MX38, MX39, MX40, MX41, MX42, MX43, MX44, MX46, MX47, MX48, MX49, MX51, MX52, MX53, MX54, MX55, MX56, MX58, MX6, MX62, MX63, MX64, MX65, MX66, MX67, MX7, MX8: footprint MX_Alps_Hybrid:MX-1U-NoLED -> MX_Only:MXOnly-1U-Hotswap
- MX14, MX19, MX45, MX5, MX50: footprint MX_Alps_Hybrid:MX-1.25U-NoLED -> MX_Only:MXOnly-1.25U-Hotswap
- MX2, MX60: footprint MX_Alps_Hybrid:MX-1.5U-NoLED -> MX_Only:MXOnly-1.5U-Hotswap
- MX3, MX4: footprint MX_Alps_Hybrid:MX-1.75U-NoLED -> MX_Only:MXOnly-1.75U-Hotswap
- MX32: footprint MX_Alps_Hybrid:MX-6.25U-NoLED -> MX_Only:MXOnly-6.25U-Hotswap
- MX57, MX61: footprint MX_Alps_Hybrid:MX-2.25U-NoLED -> MX_Only:MXOnly-2.25U-Hotswap
- MX59: footprint MX_Alps_Hybrid:MX-2U-NoLED -> MX_Only:MXOnly-2U-Hotswap
Routing:
- net ENCODER_B: track 333.5 -> 263.7 mm
- net COL2: track 127.2 -> 149.9 mm, vias 1 -> 6
- net COL6: track 121.1 -> 140.7 mm, vias 1 -> 6
- net COL3: track 104.6 -> 121.6 mm, vias 1 -> 5
- net COL1: track 144.0 -> 159.9 mm, vias 3 -> 7
- net ROW2: track 414.0 -> 399.8 mm, vias 3 -> 2
- net COL14: track 265.7 -> 279.9 mm, vias 1 -> 4
- net COL13: track 256.5 -> 269.9 mm, vias 1 -> 6
- net COL7: track 124.2 -> 136.7 mm, vias 1 -> 5
- net COL4: track 83.2 -> 95.4 mm, vias 1 -> 8
- net COL11: track 188.4 -> 199.8 mm, vias 1 -> 5
- net COL10: track 208.3 -> 219.3 mm, vias 1 -> 6
- net COL8: track 142.0 -> 152.0 mm, vias 1 -> 5
- net COL5: track 86.9 -> 96.1 mm, vias 1 -> 6
- net ROW4: track 325.5 -> 332.7 mm
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
Commit message: update kicad version
Other:
- net class Default removed
- net class Power removed
